File: powerboard1_1/powerboard1_1.sch (EAGLE design)
At the start: 106 parts, among them Q1 IPP80P03P4L04AKSA1, Q2 2N4401TFR, Q3 2N4401TFR, Q4 2N4401TFR, U1 UWQ-12/20-T48NTB-C, U2 UWE-5/20-Q48NB-C, U3 UWE-3.3/30-Q48NB-C

Commit message: Added low ESR ceramic filtering capacitors; Added open collector style on/off control circuit for each converter; Added more guideline text; Increased clearances beside Q1 to make room for optional heatsink
Parts:
- added C11, C12, C16, C17, C18, C19: (no value), rcl:C-EU025-040X050
- added C13, C14, C15, C20, C21, C22: (no value), rcl:C-EU050-035X075
- added C23, C24, C25: 100n, rcl:C-EU025-024X044
- added R15, R16: 10, rcl:R-US_0204/5
- C1: value 100u -> (none); device rcl:CPOL-USE3.5-8 -> rcl:C-EU025-040X050
- C10, C9: device rcl:CPOL-USE5-10.5 -> rcl:C-EU025-040X050
- C2, C4: value 100n -> (none); device rcl:C-EU025-024X044 -> rcl:C-EU025-040X050
- C3: value 100n -> 100u; device rcl:C-EU025-024X044 -> rcl:CPOL-USE3.5-8
- C5: device rcl:CPOL-USE2.5-7 -> rcl:C-EU025-040X050
- C6, C7: device rcl:CPOL-USE2.5-7 -> rcl:C-EU050-035X075
- C8: device rcl:CPOL-USE5-10.5 -> rcl:C-EU050-035X075
- R1: value 4.7k -> 10k
- R10, R2: value 10 -> 0.004; device rcl:R-US_0204/5 -> rcl:R-US_0617/22
- R12, R13, R14: value 0.004 -> 10; device rcl:R-US_0617/22 -> rcl:R-US_0204/5
- R3: value 10 -> 2k; device rcl:R-US_0204/5 -> resistor:R-US_0204/7
- R4: value 10 -> 4.7k; device rcl:R-US_0204/5 -> resistor:R-US_0204/7
- R5: value 2k -> 4.7k
- R6: value 36k -> 10k
- R7: value 4.7k -> 0.004; device resistor:R-US_0204/7 -> rcl:R-US_0617/22
- R8: value 4.7k -> 36k
- R9: value 10 -> 10k; device rcl:R-US_0204/5 -> resistor:R-US_0204/7
- X1: device con-phoenix-254:MPT2 -> con-phoenix-254:MPT4
Connections:
- removed net N$13: C7.+, F4.2A, F4.2B, U3.+VIN
- removed net N$9: C6.+, F3.2A, F3.2B, U2.+VIN
- removed net ON/OFF: Q2.B, Q3.B, Q4.B, R8.2, X1-2.1
- new net N$12: C16.1, C17.1, C18.1, C19.1, F4.2A, F4.2B, U3.+VIN
- new net N$7: C10.1, C11.1, C12.1, C9.1, F3.2A, F3.2B, U2.+VIN
- new net ON/OFF_1: Q2.B, R1.2, X1-4.1
- new net ON/OFF_2: Q3.B, R6.2, X1-3.1
- new net ON/OFF_3: Q4.B, R9.2, X1-2.1
- net 12V+SENSE: now also R12.2, R2.1; no longer R12.1, R9.2
- net 12V-SENSE: now also C6.1, C7.1, C8.1, PAD12.P, PAD17.P, PAD2.P, PAD37.P, PAD42.P, PAD47.P, PAD52.P, PAD55.P, PAD7.P, R11.1, R2.2; no longer C8.+, PAD23.P, PAD24.P, PAD25.P, PAD26.P, PAD28.P, PAD29.P, PAD30.P, PAD31.P, PAD33.P, R12.2, R2.1
- net 3V3+SENSE: now also R10.1, R16.2; no longer R11.2, R14.1
- net 3V3-SENSE: now also C20.1, C21.1, C22.1, PAD14.P, PAD19.P, PAD24.P, PAD29.P, PAD34.P, PAD39.P, PAD4.P, PAD44.P, PAD9.P, R10.2, R15.1; no longer C10.+, PAD46.P, PAD47.P, PAD48.P, PAD50.P, PAD51.P, PAD52.P, PAD53.P, PAD55.P, PAD56.P, R14.2, R4.1
- net 5V+SENSE: now also R14.2, R7.1; no longer R10.2, R13.1
- net 5V-SENSE: now also C13.1, C14.1, C15.1, PAD13.P, PAD18.P, PAD23.P, PAD28.P, PAD3.P, PAD33.P, PAD48.P, PAD53.P, PAD56.P, PAD8.P, R13.1, R7.2; no longer C9.+, PAD34.P, PAD35.P, PAD36.P, PAD37.P, PAD39.P, PAD40.P, PAD41.P, PAD42.P, PAD44.P, PAD45.P, R13.2, R3.1
- net GND: now also C13.2, C14.2, C15.2, C20.2, C21.2, C22.2, C6.2, C7.2, C8.2, PAD25.P, PAD26.P, PAD30.P, PAD31.P, PAD35.P, PAD36.P, PAD40.P, PAD41.P, PAD45.P, PAD46.P, PAD50.P, PAD51.P; no longer C10.-, C8.-, C9.-, PAD12.P, PAD13.P, PAD14.P, PAD17.P, PAD18.P, PAD19.P, PAD2.P, PAD3.P, PAD4.P, PAD7.P, PAD8.P, PAD9.P
- net J3: now also C25.1, R11.2; no longer C4.1, R2.2
- net J4: now also C25.2, R12.1; no longer C4.2, R9.1
- net J5: now also C24.1, R13.2; no longer C3.1, R3.2
- net J6: now also C24.2, R14.1; no longer C3.2, R10.1
- net J7: now also C23.1, R15.2; no longer C2.1, R4.2
- net J8: now also C23.2, R16.1; no longer C2.2, R11.1
- net N$1: now also R8.1; no longer R6.1
- net N$2: now also R5.2; no longer R1.2
- net N$4: now also R3.1; no longer R5.1
- net N$5: now also C1.1, C2.1, C4.1, C5.1; no longer C5.+
- net V+: now also C3.+, R4.1, R5.1, R6.1, R8.2, R9.1; no longer C1.+, R6.2, R7.1, R8.1
- net V-: now also C1.2, C10.2, C11.2, C12.2, C16.2, C17.2, C18.2, C19.2, C2.2, C3.-, C4.2, C5.2, C9.2, R3.2, R4.2; no longer C1.-, C5.-, C6.-, C7.-, R5.2, R7.2
Other:
- moved on the sheet: C2, C4, CY1, CY2, LED1, PAD1, PAD10, PAD11, PAD12, PAD13, PAD14, PAD15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

Commit message: Changed footprints of filtering capacitors and placed them closer to terminals; increased clearances between battery ground and output ground
Parts:
- added C26, C27, C28, C29, C30, C31, C32, C33, C34: (no value), rcl:C-EU025-040X050
- C1: value (none) -> 100u; device rcl:C-EU025-040X050 -> rcl:CPOL-USE3.5-8
- C10, C11, C12, C16, C5, C9: device rcl:C-EU025-040X050 -> rcl:C-EU050-035X075
- C2, C4: value (none) -> 100n; device rcl:C-EU025-040X050 -> rcl:C-EU025-024X044
- C20, C21, C22: device rcl:C-EU050-035X075 -> rcl:C-EU025-040X050
- C23, C24, C25: value 100n -> (none); device rcl:C-EU025-024X044 -> rcl:C-EU025-040X050
- C3: value 100u -> 100n; device rcl:CPOL-USE3.5-8 -> rcl:C-EU025-024X044
- R1: value 10k -> 36k
- R10: value 0.004 -> 10k; device rcl:R-US_0617/22 -> resistor:R-US_0204/7
- R14, R15, R16: value 10 -> 0.004; device rcl:R-US_0204/5 -> rcl:R-US_0617/22
- R2, R7: value 0.004 -> 4.7k; device rcl:R-US_0617/22 -> resistor:R-US_0204/7
- R3: value 2k -> 10; device resistor:R-US_0204/7 -> rcl:R-US_0204/5
- R4, R5: value 4.7k -> 10; device resistor:R-US_0204/7 -> rcl:R-US_0204/5
- R6: value 10k -> 2k
- R8: value 36k -> 10k
Connections:
- net 12V+SENSE: now also C17.1, C18.1, C23.1, C24.1, C29.1, C30.1, R11.2, R14.1; no longer R12.2, R2.1
- net 12V-SENSE: now also PAD23.P, PAD24.P, PAD25.P, PAD26.P, PAD28.P, PAD29.P, PAD30.P, PAD31.P, PAD33.P, R14.2, R3.1; no longer C6.1, C7.1, C8.1, PAD12.P, PAD17.P, PAD2.P, PAD37.P, PAD42.P, PAD47.P, PAD52.P, PAD55.P, PAD7.P, R11.1, R2.2
- net 3V3+SENSE: now also C21.1, C22.1, C27.1, C28.1, C33.1, C34.1, R13.2, R16.1; no longer R10.1, R16.2
- net 3V3-SENSE: now also PAD46.P, PAD47.P, PAD48.P, PAD50.P, PAD51.P, PAD52.P, PAD53.P, PAD55.P, PAD56.P, R16.2, R5.1; no longer C20.1, C21.1, C22.1, PAD14.P, PAD19.P, PAD24.P, PAD29.P, PAD34.P, PAD39.P, PAD4.P, PAD44.P, PAD9.P, R10.2, R15.1
- net 5V+SENSE: now also C19.1, C20.1, C25.1, C26.1, C31.1, C32.1, R12.2, R15.1; no longer R14.2, R7.1
- net 5V-SENSE: now also PAD34.P, PAD35.P, PAD36.P, PAD37.P, PAD39.P, PAD40.P, PAD41.P, PAD42.P, PAD44.P, PAD45.P, R15.2, R4.1; no longer C13.1, C14.1, C15.1, PAD13.P, PAD18.P, PAD23.P, PAD28.P, PAD3.P, PAD33.P, PAD48.P, PAD53.P, PAD56.P, PAD8.P, R13.1, R7.2
- net GND: now also C17.2, C18.2, C19.2, C23.2, C24.2, C25.2, C26.2, C27.2, C28.2, C29.2, C30.2, C31.2, C32.2, C33.2, C34.2, PAD12.P, PAD13.P, PAD14.P, PAD17.P, PAD18.P, PAD19.P, PAD2.P, PAD3.P, PAD4.P, PAD7.P, PAD8.P, PAD9.P; no longer C13.2, C14.2, C15.2, C6.2, C7.2, C8.2, PAD25.P, PAD26.P, PAD30.P, PAD31.P, PAD35.P, PAD36.P, PAD40.P, PAD41.P, PAD45.P, PAD46.P, PAD50.P, PAD51.P
- net J3: now also C4.1, R3.2; no longer C25.1, R11.2
- net J4: now also C4.2, R11.1; no longer C25.2, R12.1
- net J5: now also C3.1, R4.2; no longer C24.1, R13.2
- net J6: now also C3.2, R12.1; no longer C24.2, R14.1
- net J7: now also C2.1, R5.2; no longer C23.1, R15.2
- net J8: now also C2.2, R13.1; no longer C23.2, R16.1
- net N$1: now also R1.1; no longer R8.1
- net N$12: now also C10.1, C15.1, C9.1; no longer C17.1, C18.1, C19.1
- net N$2: now also R2.2; no longer R5.2
- net N$4: now also R6.1; no longer R3.1
- net N$5: now also C11.1, C12.1, C6.1; no longer C1.1, C2.1, C4.1
- net N$7: now also C13.1, C14.1, C7.1, C8.1; no longer C10.1, C11.1, C12.1, C9.1
- net ON/OFF_1: now also R8.2; no longer R1.2
- net ON/OFF_2: now also R9.2; no longer R6.2
- net ON/OFF_3: now also R10.2; no longer R9.2
- net V+: now also C1.+, R1.2, R10.1, R2.1, R7.1, R8.1; no longer C3.+, R1.1, R4.1, R5.1, R6.1, R8.2
- net V-: now also C1.-, C13.2, C14.2, C15.2, C6.2, C7.2, C8.2, R6.2, R7.2; no longer C1.2, C17.2, C18.2, C19.2, C2.2, C3.-, C4.2, R3.2, R4.2
Other:
- moved on the sheet: C10, C11, C12, C13, C14, C15, C16, C17, C18, C19, C2, C20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
