File: Battery Voltage Monitoring Schematic.sch (EAGLE design)
At the start: 13 parts, among them U1 INA3221.

Commit message: Add files via upload
Parts:
- removed JP1, JP2: (no value), pinhead:PINHD-1X14
- added R3: (no value), rcl:R-US_R0805
- added U$1: TEENSY_3.1-3.2_OUTER_ROW, Teensy_3_and_LC_Series_Boards_v1.4:TEENSY_3.1-3.2_OUTER_ROW
- added U2: INA3221., INA3221:INA3221.
- added X1: (no value), con-molex:KK-156-16
- C3: value (none) -> 0.1microF
- R10, R2, R5, R6, R8, R9: value (none) -> 10kOhm
Connections:
- removed net LCD_ENABLE: JP2.14
- removed net LCD_RS: JP2.13
- new net 0-26V_BATTERY4: R7.2, U2.IN+2
- new net 14/A0: U$1.14/A0, X1-4.S
- new net LCD_DB4: U$1.23/A9/T/PWM, X1-11.S
- new net SCK(LED): U$1.13/SCK/LED, X1-6.S
- net 0-26V_BATTERY3: now also R3.2, U2.IN+1; no longer R2.2, U1.IN+3
- net 3.3V: now also U$1.3.3V, U2.VS; no longer JP2.3
- net 5V: now also U$1.VIN, X1-15.S, X1-2.S; no longer JP2.1
- net CRITICAL_OUT: now also R8.1, U$1.9/RX2/PWM, U2.CRITICAL; no longer JP1.11, R9.1
- net GND: now also R3.1, R7.1, U$1.GND, U1.A0, U2.GND, U2.IN-1, U2.IN-2, X1-1.S, X1-16.S, X1-5.S; no longer JP1.1, R2.1, U1.IN-3
- net LCD_DB5: now also U$1.22/A8/T/PWM, X1-12.S; no longer JP2.5
- net LCD_DB6: now also U$1.21/A7/PWM, X1-13.S; no longer JP2.6
- net LCD_DB7: now also U$1.20/A6/PWM, X1-14.S; no longer JP2.7
- net PV_OUT: now also R2.2, U$1.7/RX3, U2.PV; no longer JP1.9, R7.2
- net SDA_OUT: now also R6.1, U$1.17/A3/T, U2.SDA; no longer JP2.10, R5.1
- net TC_OUT: now also R9.1, U$1.8/TX3, U2.TC; no longer JP1.10, R10.1
- net TEENSY_SCK: now also R5.1, U$1.16/A2/T, U2.SCL; no longer JP2.11, R6.1
- net VPU: now also R2.1, U2.VPU; no longer R7.1
- net WARNING_OUT: now also R10.1, U$1.10/TX2/PWM, U2.WARNING; no longer JP1.12, R8.1
Other:
- note added: "potentiometer between Vdd and Vss with middle pin to V0"
- note added: "to LCD_RS"
- note added: "to LCD_enable"
- note removed: "0.1microF"
- note removed: "Teensy"
- note removed: "suggested 10kOhm"
- note removed: "to OUT DRV5033"
- note removed: "to VCC DRV5033"
- moved on the sheet: C3, R1, R10, R2, R4, R5, R6, R7, R8, R9

Commit message: Add files via upload
Parts:
- added C1: 0.1microF, rcl:C-USC0805
- added IC1: 74HC595N, 74xx-eu:74HC595N
Connections:
- new net ENABLE: IC1A.QD, X1-6.S
- new net N$3: IC1A.QA
- new net N$5: IC1A.QC
- new net RS: IC1A.QB, X1-4.S
- new net SER: IC1A.SER, U$1.11/MOSI
- net 14/A0: no longer X1-4.S
- net 5V: now also C1.1, IC1A.SCL, IC1P.VCC
- net GND: now also C1.2, IC1A.G, IC1P.GND
- net LCD_DB4: now also IC1A.QE; no longer U$1.23/A9/T/PWM
- net LCD_DB5: now also IC1A.QF; no longer U$1.22/A8/T/PWM
- net LCD_DB6: now also IC1A.QG; no longer U$1.21/A7/PWM
- net LCD_DB7: now also IC1A.QH; no longer U$1.20/A6/PWM
- net SCK(LED): now also IC1A.RCK, IC1A.SCK; no longer X1-6.S
Other:
- moved on the sheet: X1-1, X1-10, X1-11, X1-12, X1-13, X1-14, X1-15, X1-16, X1-2, X1-3, X1-4, X1-5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

Commit message: Add files via upload
Parts:
- removed C3: 0.1microF, rcl:C-USC0805
- added C2, C4: 0.1microF, rcl:C-USC0805
- added R11, R12, R13, R14, R15, R16: 560Ohm, rcl:R-US_R0805
Connections:
- net 3.3V: now also C4.1; no longer C3.1
- net ENABLE: now also R12.1
- net GND: now also C2.2, C4.2, U1.IN-3, U2.IN-3; no longer C3.2
- net LCD_DB4: now also R13.1, R13.2
- net LCD_DB5: now also R14.2
- net LCD_DB6: now also R15.1, R15.2
- net LCD_DB7: now also R16.1
- net RS: now also R11.1, R11.2
Other:
- note added: "R>1936Ohm"
- moved on the sheet: C1

Commit message: Add files via upload
Parts:
- removed U$1: TEENSY_3.1-3.2_OUTER_ROW, Teensy_3_and_LC_Series_Boards_v1.4:TEENSY_3.1-3.2_OUTER_ROW
- added DIS1: TUXGR_16X2_R2, display-lcd:TUXGR_16X2_R2
- added J1: 22-27-2031-03, con-molex:22-27-2031-03
- added PAD10_M1, PAD11_GND, PAD12_M2, PAD13_GND, PAD14_M3, PAD15_GND, PAD16_M4, PAD1_GND, PAD2_B1, PAD3_GND, PAD4_B2, PAD5_GND, PAD6_B3, PAD7_GND, PAD8_B4, PAD9_GND: 3,81/1,9, Moira:3,81/1,9
- added R22: 10kOhm, pot:TRIM_US-SM-42/43W
- added U$14: TEENSY_3.1-3.2_DIL, Teensy_3_and_LC_Series_Boards_v1.4:TEENSY_3.1-3.2_DIL
- added X3: 2516-, con-3m:2516-
- C1, C2, C4: device rcl:C-USC0805 -> resistor:C-USC2012
- IC1: value 74HC595N -> 74HC595D; device 74xx-eu:74HC595N -> 74xx-eu:74HC595D
- R1, R3, R4, R7: value (none) -> 0.001Ohm; device rcl:R-US_R0805 -> Moira:HCS3920FT1L00
- R10, R11, R12, R13, R14, R15, R16, R2, R5, R6, R8, R9: device rcl:R-US_R0805 -> rcl:R-US_M2012
- X1: value (none) -> 22-27-2021-02; device con-molex:KK-156-16 -> con-molex:22-27-2021-02
Connections:
- removed net 14/A0: U$1.14/A0
- removed net 5V: C1.1, IC1A.SCL, IC1P.VCC, U$1.VIN, X1-15.S, X1-2.S
- removed net N$3: IC1A.QA
- removed net N$5: IC1A.QC
- removed net SCK(LED): IC1A.RCK, IC1A.SCK, U$1.13/SCK/LED
- removed net SER: IC1A.SER, U$1.11/MOSI
- removed net VPU: R2.1, U1.VPU, U2.VPU
- new net +5V: C1.1, DIS1.VCC, IC1A.SCL, IC1P.VCC, R22.A, U$14.VIN, X1-1.S, X3-2.KL
- new net AGND: PAD11_GND.P, PAD13_GND.P, PAD15_GND.P, PAD1_GND.P, PAD3_GND.P, PAD5_GND.P, PAD7_GND.P, PAD9_GND.P, X3-4.KL
- new net BACKLIGHT: DIS1.NC@1, U$14.3/CAN-TX/PWM, X3-3.KL
- new net DATA: IC1A.SER, U$14.11/MOSI, X3-15.KL
- new net ENABLE1: IC1A.QG, R12.1
- new net HALL: J1-3.S, U$14.5/PWM, X3-5.KL
- new net LATCH: IC1A.RCK, U$14.14/A1, X3-12.KL
- new net LCD(SCK): IC1A.SCK, U$14.13/SCK/LED, X3-14.KL
- new net LCD_DB41: IC1A.QD, R13.1
- new net LCD_DB51: IC1A.QC, R14.1
- new net LCD_DB61: IC1A.QB, R15.1
- new net LCD_DB71: IC1A.QA, R16.2
- new net MOTOR1: PAD10_M1.P, R4.1, U1.IN-1
- new net MOTOR2: PAD12_M2.P, R1.1, U1.IN-2, U1.IN-3
- new net MOTOR3: PAD14_M3.P, R3.1, U2.IN-1
- new net MOTOR4: PAD16_M4.P, R7.1, U2.IN-2, U2.IN-3
- new net N$18: DIS1.CONTR, R22.S
- new net RS1: IC1A.QH, R11.1
- net 0-26V_BATTERY1: now also PAD2_B1.P
- net 0-26V_BATTERY2: now also PAD4_B2.P
- net 0-26V_BATTERY3: now also PAD6_B3.P
- net 0-26V_BATTERY4: now also PAD8_B4.P
- net 3.3V: now also C2.1, J1-1.S, R2.1, U$14.3.3V, U1.VPU, U2.A0, U2.VPU, X3-6.KL; no longer U$1.3.3V
- net CRITICAL_OUT: now also U$14.9/RX2/PWM, X3-11.KL; no longer U$1.9/RX2/PWM
- net ENABLE: now also DIS1.E, R12.2; no longer IC1A.QD, R12.1, X1-6.S
- net GND: now also DIS1.GND, DIS1.NC@2, DIS1.R/W, IC1A.QF, J1-2.S, R22.E, U$14.GND, X1-2.S, X3-1.KL; no longer R1.1, R3.1, R4.1, R7.1, U$1.GND, U1.IN-1, U1.IN-2, U1.IN-3, U2.IN-1, U2.IN-2, U2.IN-3, X1-1.S, X1-16.S, X1-5.S
- net LCD_DB4: now also DIS1.D4; no longer IC1A.QE, R13.1, X1-11.S
- net LCD_DB5: now also DIS1.D5; no longer IC1A.QF, X1-12.S
- net LCD_DB6: now also DIS1.D6; no longer IC1A.QG, R15.1, X1-13.S
- net LCD_DB7: now also DIS1.D7; no longer IC1A.QH, X1-14.S
- net PV_OUT: now also U$14.7/RX3, X3-7.KL; no longer U$1.7/RX3
- net RS: now also DIS1.RS; no longer IC1A.QB, R11.1, X1-4.S
- net SDA_OUT: now also U$14.18/A4/T/SDA0, X3-10.KL; no longer U$1.17/A3/T
- net TC_OUT: now also U$14.8/TX3, X3-9.KL; no longer U$1.8/TX3
- net TEENSY_SCK: now also U$14.19/A5/T/SCL0, X3-8.KL; no longer U$1.16/A2/T
- net WARNING_OUT: now also U$14.10/TX2/PWM, X3-13.KL; no longer U$1.10/TX2/PWM
Other:
- note added: "14 guage, power and ground, 4 across the top for the batteries"
- note added: "3.3V"
- note removed: "Kelvin connection?"
- note removed: "Load?"
- note removed: "R>1936Ohm"
- note removed: "potentiometer between Vdd and Vss with middle pin to V0"
- note removed: "to LCD_RS"
- note removed: "to LCD_enable"
- moved on the sheet: C1, C4, IC1, IC1P, R10, R11, R12, R13, R14, R15, R16, R2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

Commit message: Add files via upload
Parts:
- removed PAD10_M1, PAD11_GND, PAD12_M2, PAD13_GND, PAD14_M3, PAD15_GND, PAD16_M4, PAD1_GND, PAD2_B1, PAD3_GND, PAD4_B2, PAD5_GND, PAD6_B3, PAD7_GND, PAD8_B4, PAD9_GND: 3,81/1,9, Moira:3,81/1,9
- removed X1: 22-27-2021-02, con-molex:22-27-2021-02
- added U$1, U$2, U$3, U$4, U$5, U$6, U$7, U$8: MKDS_5/2-6,352, Moira:MKDS_5/2-6,352
- added U$10: ARVP_LOGO, ARVP:ARVP_LOGO
- added U$9: ARVP_MOLEX_FEMALE, ARVP_MOLEX_FEMALE:ARVP_MOLEX_FEMALE
Connections:
- net +5V: now also U$9.P$1; no longer X1-1.S
- net 0-26V_BATTERY1: now also U$1.KL; no longer PAD2_B1.P
- net 0-26V_BATTERY2: now also U$2.KL; no longer PAD4_B2.P
- net 0-26V_BATTERY3: now also U$3.KL; no longer PAD6_B3.P
- net 0-26V_BATTERY4: now also U$4.KL; no longer PAD8_B4.P
- net AGND: now also U$1.KL1, U$2.KL1, U$3.KL1, U$4.KL1, U$5.KL1, U$6.KL1, U$7.KL1, U$8.KL1; no longer PAD11_GND.P, PAD13_GND.P, PAD15_GND.P, PAD1_GND.P, PAD3_GND.P, PAD5_GND.P, PAD7_GND.P, PAD9_GND.P
- net GND: now also U$9.P$2; no longer X1-2.S
- net MOTOR1: now also U$5.KL; no longer PAD10_M1.P
- net MOTOR2: now also U$6.KL; no longer PAD12_M2.P
- net MOTOR3: now also U$7.KL; no longer PAD14_M3.P
- net MOTOR4: now also U$8.KL; no longer PAD16_M4.P

Commit message: Add files via upload
Battery AGND connected to teensy GND
Connections:
- net AGND: no longer U$4.KL1
- net GND: now also U$4.KL1
Changed lines of the file:
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@@
 <part name="U$9" library="ARVP_MOLEX_FEMALE" deviceset="ARVP_MOLEX_FEMALE" device=""/>
 <part name="U$10" library="ARVP" deviceset="ARVP_LOGO" device=""/>
+<part name="GND14" library="supply1" deviceset="GND" device=""/>
 </parts>
 <sheets>
@@
 <instance part="U$9" gate="G$1" x="91.44" y="182.88" rot="R90"/>
 <instance part="U$10" gate="G$1" x="91.44" y="55.88"/>
+<instance part="GND14" gate="1" x="73.66" y="81.28"/>
 </instances>
 <busses>
@@
 <wire x1="170.18" y1="-43.18" x2="170.18" y2="-40.64" width="0.1524" layer="91"/>
 <pinref part="GND2" gate="1" pin="GND"/>
+</segment>
+<segment>
+<pinref part="GND18" gate="VR1" pin="AGND"/>
+<pinref part="U$4" gate="G$1" pin="KL1"/>
+<wire x1="73.66" y1="91.44" x2="73.66" y2="96.52" width="0.1524" layer="91"/>
+<wire x1="73.66" y1="91.44" x2="73.66" y2="83.82" width="0.1524" layer="91"/>
+<junction x="73.66" y="91.44"/>
+<pinref part="GND14" gate="1" pin="GND"/>
 </segment>
 </net>
@@
 <net name="AGND" class="0">
 <segment>
+<pinref part="GND16" gate="VR1" pin="AGND"/>
+<pinref part="U$2" gate="G$1" pin="KL1"/>
+<wire x1="45.72" y1="91.44" x2="45.72" y2="96.52" width="0.1524" layer="91"/>
+</segment>
+<segment>
+<pinref part="GND17" gate="VR1" pin="AGND"/>
+<pinref part="U$3" gate="G$1" pin="KL1"/>
+<wire x1="58.42" y1="91.44" x2="58.42" y2="96.52" width="0.1524" layer="91"/>
+</segment>
+<segment>
+<pinref part="GND19" gate="VR1" pin="AGND"/>
+<pinref part="U$5" gate="G$1" pin="KL1"/>
+<wire x1="71.12" y1="-40.64" x2="71.12" y2="-45.72" width="0.1524" layer="91"/>
+</segment>
+<segment>
+<pinref part="GND20" gate="VR1" pin="AGND"/>
+<pinref part="U$6" gate="G$1" pin="KL1"/>
+<wire x1="83.82" y1="-40.64" x2="83.82" y2="-45.72" width="0.1524" layer="91"/>
+</segment>
+<segment>
+<pinref part="GND21" gate="VR1" pin="AGND"/>
+<pinref part="U$7" gate="G$1" pin="KL1"/>
+<wire x1="96.52" y1="-40.64" x2="96.52" y2="-45.72" width="0.1524" layer="91"/>
+</segment>
+<segment>
+<pinref part="GND22" gate="VR1" pin="AGND"/>
+<pinref part="U$8" gate="G$1" pin="KL1"/>
+<wire x1="109.22" y1="-40.64" x2="109.22" y2="-45.72" width="0.1524" layer="91"/>
+</segment>
+<segment>
+<pinref part="X3" gate="-4" pin="KL"/>
+<wire x1="177.8" y1="-43.18" x2="177.8" y2="-40.64" width="0.1524" layer="91"/>
+<pinref part="GND11" gate="VR1" pin="AGND"/>
+</segment>
+<segment>
 <pinref part="AGND" gate="VR1" pin="AGND"/>
 <pinref part="U$1" gate="G$1" pin="KL1"/>
 <wire x1="33.02" y1="91.44" x2="33.02" y2="96.52" width="0.1524" layer="91"/>
 </segment>
-<segment>
-<pinref part="GND16" gate="VR1" pin="AGND"/>
-<pinref part="U$2" gate="G$1" pin="KL1"/>
-<wire x1="45.72" y1="91.44" x2="45.72" y2="96.52" width="0.1524" layer="91"/>
-</segment>
-<segment>
-<pinref part="GND17" gate="VR1" pin="AGND"/>
-<pinref part="U$3" gate="G$1" pin="KL1"/>
-<wire x1="58.42" y1="91.44" x2="58.42" y2="96.52" width="0.1524" layer="91"/>
-</segment>
-<segment>
-<pinref part="GND18" gate="VR1" pin="AGND"/>
-<pinref part="U$4" gate="G$1" pin="KL1"/>
-<wire x1="73.66" y1="91.44" x2="73.66" y2="96.52" width="0.1524" layer="91"/>
-</segment>
-<segment>
-<pinref part="GND19" gate="VR1" pin="AGND"/>
-<pinref part="U$5" gate="G$1" pin="KL1"/>
-<wire x1="71.12" y1="-40.64" x2="71.12" y2="-45.72" width="0.1524" layer="91"/>
-</segment>
-<segment>
-<pinref part="GND20" gate="VR1" pin="AGND"/>
-<pinref part="U$6" gate="G$1" pin="KL1"/>
-<wire x1="83.82" y1="-40.64" x2="83.82" y2="-45.72" width="0.1524" layer="91"/>
-</segment>
-<segment>
-<pinref part="GND21" gate="VR1" pin="AGND"/>
-<pinref part="U$7" gate="G$1" pin="KL1"/>
-<wire x1="96.52" y1="-40.64" x2="96.52" y2="-45.72" width="0.1524" layer="91"/>
-</segment>
-<segment>
-<pinref part="GND22" gate="VR1" pin="AGND"/>
-<pinref part="U$8" gate="G$1" pin="KL1"/>
-<wire x1="109.22" y1="-40.64" x2="109.22" y2="-45.72" width="0.1524" layer="91"/>
-</segment>
-<segment>
-<pinref part="X3" gate="-4" pin="KL"/>
-<wire x1="177.8" y1="-43.18" x2="177.8" y2="-40.64" width="0.1524" layer="91"/>
-<pinref part="GND11" gate="VR1" pin="AGND"/>
-</segment>
-</net>
+</net>

Commit message: Changed terminal block layout; Modified some routing; Fixed DRC issues
Parts:
- removed DIS1: TUXGR_16X2_R2, display-lcd:TUXGR_16X2_R2
- removed U$8: MKDS_5/2-6,352, Moira:MKDS_5/2-6,352
- added JP1: (no value), pinhead:PINHD-1X16
- added U$11: MKDS_5/2-6,352, Moira:MKDS_5/2-6,352
Connections:
- net +5V: now also JP1.2; no longer DIS1.VCC
- net AGND: no longer U$1.KL1, U$2.KL1, U$3.KL1, U$5.KL1, U$6.KL1, U$7.KL1, U$8.KL1
- net BACKLIGHT: now also JP1.15; no longer DIS1.NC@1
- net ENABLE: now also JP1.6; no longer DIS1.E
- net GND: now also JP1.1, JP1.16, JP1.5, U$1.KL1, U$11.KL, U$2.KL1, U$3.KL1, U$5.KL, U$6.KL, U$7.KL; no longer DIS1.GND, DIS1.NC@2, DIS1.R/W
- net LCD_DB4: now also JP1.11; no longer DIS1.D4
- net LCD_DB5: now also JP1.12; no longer DIS1.D5
- net LCD_DB6: now also JP1.13; no longer DIS1.D6
- net LCD_DB7: now also JP1.14; no longer DIS1.D7
- net MOTOR1: now also U$7.KL1; no longer U$5.KL
- net MOTOR2: now also U$6.KL1; no longer U$6.KL, U1.IN-3
- net MOTOR3: now also U$5.KL1; no longer U$7.KL
- net MOTOR4: now also U$11.KL1; no longer U$8.KL, U2.IN-3
- net N$18: now also JP1.3; no longer DIS1.CONTR
- net RS: now also JP1.4; no longer DIS1.RS
Other:
- moved on the sheet: U$5, U$7
