File: Battery_Monitoring_with_kill_Schematic.sch (EAGLE design)
At the start: 60 parts, among them CON2 MOLEX_5566-2, U1 INA3221., U2 INA3221., U5 TEENSY_3.1_BASIC_2, U6 TCAN1042HVDR, X2 OSTVN02A150

Commit message: Fixed GND's and removed AGND's
Parts:
- removed CON2: MOLEX_5566-2, ARVP:MOLEX_5566-2
- removed JP4: (no value), pinhead:PINHD-2X3
- removed JP5: (no value), pinhead:PINHD-1X2
- removed JP6: (no value), pinhead:PINHD-2X4
- removed R14, R15, R21: 1, adafruit:R-US_M1206
- removed R17: 220, rcl:R-US_R0805
- removed R18, R19: 10k, rcl:R-US_R1206
- removed R2, R5: 10kOhm, rcl:R-US_M2012
- removed R20: 1k, rcl:R-US_R0805
- removed U$9: ARVP_MOLEX_FEMALE, ARVP_MOLEX_FEMALE:ARVP_MOLEX_FEMALE
- removed U5: TEENSY_3.1_BASIC_2, Teensy_3_Series_Board_v1.0:TEENSY_3.1_BASIC_2
- removed X2: OSTVN02A150, dropper_torpedo_v3:OSTVN02A150
- added CON4: MOLEX_5566-2, ARVP:MOLEX_5566-2
- added CON5, CON6: S3B-PH-SM4-TB, ARVP:S3B-PH-SM4-TB
- added JP1: (no value), pinhead:PINHD-2X3
- added JP2: (no value), pinhead:PINHD-1X2
- added JP3: (no value), pinhead:PINHD-2X4
- added U4: TEENSY_3.1_BASIC_2, Teensy_3_Series_Board_v1.0:TEENSY_3.1_BASIC_2
- R10, R9: value 10kOhm -> 10k; device rcl:R-US_M2012 -> rcl:R-US_R1206
- R16: value 220 -> 1k
- R6, R8: value 10kOhm -> 220; device rcl:R-US_M2012 -> rcl:R-US_R0805
Connections:
- removed net AGND: R14.2, R15.2, R21.2, U$1.KL1, U$2.KL1, U$3.KL1, U$5.KL1, U$6.KL1, U$7.KL1, U$8.KL1
- removed net CAN_TX1: R16.2, U6.TXD
- removed net I2_3V1: JP4.6, JP6.7, JP6.8
- removed net PCA_OE: U5.11/MOSI
- removed net SDA_OUT: JP6.5, JP6.6, R18.2, R6.1, U1.SDA, U2.SDA, U5.18/A4/T/SDA0
- removed net TEENSY_SCK: JP6.3, JP6.4, R19.2, R5.1, U1.SCL, U2.SCL, U5.19/A5/T/SCL0
- removed net TRP0: U5.16/A2/T
- removed net TRP1: U5.17/A3/T
- new net CANSH1: CON5-1.S, CON6-1.S
- new net CAN_TX2: R6.2, U6.TXD
- new net I2C_3V1: JP1.6, JP3.7, JP3.8
- new net SCL: JP3.5, JP3.6, R10.2, U1.SCL, U2.SCL, U4.19/A5/T/SCL0
- new net SDA: JP3.3, JP3.4, R9.2, U1.SDA, U2.SDA, U4.18/A4/T/SDA0
- net +3V3: now also JP1.1, JP1.3, JP1.5, U4.3.3V; no longer JP4.1, JP4.3, JP4.5, U5.3.3V
- net +5V: now also CON4G$1.S, JP2.2; no longer CON2G$1.S, JP5.2, U$9.P$1
- net 3.3V: no longer R10.2, R2.1, R5.2, R6.2, R8.2, R9.2
- net CANH1: now also CON5-3.S, CON6-3.S; no longer X2G$2.1
- net CANL1: now also CON5-2.S, CON6-2.S; no longer X2G$1.1
- net CAN_RX1: now also R8.2; no longer R17.2
- net CAN_RX_T: now also R8.1, U4.4/CAN-RX-PWM; no longer R17.1, U5.4/CAN-RX-PWM
- net CAN_TX_T: now also R6.1, U4.3/CAN-TX/PWM; no longer R16.1, U5.3/CAN-TX/PWM
- net CRITICAL_OUT: now also U4.9/RX2/PWM; no longer R8.1, U5.9/RX2/PWM
- net GND: now also CON4G$2.S, CON5-TABS.S, CON6-TABS.S, JP3.1, JP3.2, R16.1, U$1.KL1, U$2.KL1, U$3.KL1, U$8.KL1, U4.GND; no longer CON2G$2.S, JP6.1, JP6.2, R20.1, U$9.P$2, U5.GND
- net MD1: now also U$5.KL1; no longer R14.1
- net MD2: now also U$6.KL1; no longer R15.1
- net MD3: now also U$7.KL1; no longer R21.1
- net PV_OUT: now also U4.7/RX3; no longer R2.2, U5.7/RX3
- net SCL_3V1: now also JP1.2, R10.1; no longer JP4.2, R19.1
- net SDA_3V1: now also JP1.4, R9.1; no longer JP4.4, R18.1
- net STB1: now also R16.2; no longer R20.2
- net TC_OUT: now also U4.8/TX3; no longer R9.1, U5.8/TX3
- net VIN: now also JP2.1, U4.VIN; no longer JP5.1, U5.VIN
- net WARNING_OUT: now also U4.10/TX2/PWM; no longer R10.1, U5.10/TX2/PWM
Other:
- note added: "to SCL PIN"
- note added: "to SDA PIN"
- note removed: "14 guage, power and ground, 4 across the top for the batteries"
- note removed: "INA3221 Pullups"
- moved on the sheet: C5, C6, R10, R16, R6, R8, R9, U6

Commit message: Added jumpers to schematic and finished the PCB. The PCB has not been checked with the new DRC.
Parts:
- removed J1: (no value), SparkFun-Connectors:CONN_03
- added JP4, JP5: (no value), pinhead:PINHD-1X2
- added JP6: (no value), pinhead:PINHD-1X3
Connections:
- removed net 3.3V: C2.1, C4.1, U1.VPU, U1.VS, U2.A0, U2.VPU, U2.VS
- new net N$5: JP5.2, JP6.2
- net +3V3: now also C2.1, C4.1, U1.VPU, U1.VS, U2.A0, U2.VPU, U2.VS
- net +5V: now also JP6.1; no longer J1.1
- net GND: now also JP4.2, JP6.3; no longer J1.3
- net N$4: now also JP4.1, JP5.1; no longer J1.2
Other:
- note added: "Bypass Jumper"
- note added: "Mechanical Kill"
