File: communications_hub/communication-hub/i2c_board.sch (EAGLE design)
At the start: 40 parts, among them CON3 SM03B-GHS-TB, CON4 SM03B-GHS-TB, U3 TCAN1042HVDR, U4 TCAN1042HVDR

Commit message: Fine tuned positions of 30 and 40 pin headers
Parts:
- J21: device pinhead:PINHD-2X20 -> commhub:PINHD-2X20
- J26: device pinhead:PINHD-2X15 -> commhub:PINHD-2X15
Changed lines of the file:
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@@
 <?xml version="1.0" encoding="utf-8"?>
 <!DOCTYPE eagle SYSTEM "eagle.dtd">
-<eagle version="8.3.2">
+<eagle version="8.4.1">
 <drawing>
 <settings>
@@
 <layers>
 <layer number="1" name="Top" color="4" fill="1" visible="no" active="no"/>
+<layer number="2" name="Route2" color="1" fill="3" visible="no" active="no"/>
+<layer number="3" name="Route3" color="4" fill="3" visible="no" active="no"/>
+<layer number="4" name="Route4" color="1" fill="4" visible="no" active="no"/>
+<layer number="5" name="Route5" color="4" fill="4" visible="no" active="no"/>
+<layer number="6" name="Route6" color="1" fill="8" visible="no" active="no"/>
+<layer number="7" name="Route7" color="4" fill="8" visible="no" active="no"/>
+<layer number="8" name="Route8" color="1" fill="2" visible="no" active="no"/>
+<layer number="9" name="Route9" color="4" fill="2" visible="no" active="no"/>
+<layer number="10" name="Route10" color="1" fill="7" visible="no" active="no"/>
+<layer number="11" name="Route11" color="4" fill="7" visible="no" active="no"/>
+<layer number="12" name="Route12" color="1" fill="5" visible="no" active="no"/>
+<layer number="13" name="Route13" color="4" fill="5" visible="no" active="no"/>
+<layer number="14" name="Route14" color="1" fill="6" visible="no" active="no"/>
+<layer number="15" name="Route15" color="4" fill="6" visible="no" active="no"/>
 <layer number="16" name="Bottom" color="1" fill="1" visible="no" active="no"/>
 <layer number="17" name="Pads" color="2" fill="1" visible="no" active="no"/>
@@
 </classes>
 <parts>
-<part name="J21" library="pinhead" library_urn="urn:adsk.eagle:library:325" deviceset="PINHD-2X20" device="" package3d_urn="urn:adsk.eagle:package:22443/2"/>
-<part name="J26" library="pinhead" library_urn="urn:adsk.eagle:library:325" deviceset="PINHD-2X15" device="" package3d_urn="urn:adsk.eagle:package:22427/1"/>
+<part name="J21" library="commhub" deviceset="PINHD-2X20" device=""/>
+<part name="J26" library="commhub" deviceset="PINHD-2X15" device=""/>
 <part name="U$3" library="molex-sl-connectors_jw" deviceset="MOLEX_SL_02" device="-70553"/>
 <part name="U$4" library="molex-sl-connectors_jw" deviceset="MOLEX_SL_04" device="-70553"/>

Commit message: Finished first revision of communication hub board. Needs to be reviewed before commit.
Parts:
- removed U$3: MOLEX_SL_02-70553, molex-sl-connectors_jw:MOLEX_SL_02-70553
- removed U$4, U$5: MOLEX_SL_04-70553, molex-sl-connectors_jw:MOLEX_SL_04-70553
- added CON1, CON2: SM04B-GHS-TB, ARVP:SM04B-GHS-TB
- added CON5: SM02B-GHS-TB, ARVP:SM02B-GHS-TB
- JP5: device jumper:JP2Q -> jumper:JP1Q
Connections:
- net +3V3: now also J21.1, JP1.2, JP2.2, JP5.2; no longer JP5.3
- net +5V: now also J21.2
- net CAN0_TX_T: now also J26.7
- net CAN1_TX_T: no longer J26.7
- net GND: now also CON1-1.S, CON2-1.S, J21.14, J21.20, J21.25, J21.30, J21.34, J21.35, J21.6, J21.9; no longer U$4.4, U$5.4
- net I2C_GP0_SCL: now also CON2-3.S; no longer U$4.2
- net I2C_GP0_SDA: now also CON2-2.S; no longer U$4.3
- net I2C_GP1_SCL: now also CON1-3.S; no longer U$5.2
- net I2C_GP1_SDA: now also CON1-2.S; no longer U$5.3
- net N$6: now also CON1-4.S, CON2-4.S; no longer U$4.1, U$5.1
- net UART1_RX: now also CON5-2.S; no longer U$3.1
- net UART1_TX: now also CON5-1.S; no longer U$3.2
Other:
- note added: "Expansion Header"
- note added: "GPIO Header"

Commit message: Made requisite changes to communications hub.
Parts:
- added JP6: (no value), jumper:JP1Q
- renumbered LED3 to LED1, LED4 to LED2
Connections:
- new net N$5: CON1-4.S, JP6.1
- net +3V3: now also JP6.2
- net N$6: no longer CON1-4.S
Other:
- moved on the sheet: CON1-TABS, CON2-TABS, JP5
Changed lines of the file:
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@@
 <part name="R10" library="resistor" library_urn="urn:adsk.eagle:library:348" deviceset="R-US_" device="M1206" package3d_urn="urn:adsk.eagle:package:26088/1"/>
 <part name="+3V10" library="supply1" library_urn="urn:adsk.eagle:library:371" deviceset="+3V3" device=""/>
-<part name="LED3" library="eagle-ltspice" library_urn="urn:adsk.eagle:library:217" deviceset="LED_E" device="" package3d_urn="urn:adsk.eagle:package:13319/1"/>
-<part name="LED4" library="eagle-ltspice" library_urn="urn:adsk.eagle:library:217" deviceset="LED_E" device="" package3d_urn="urn:adsk.eagle:package:13319/1"/>
+<part name="LED1" library="eagle-ltspice" library_urn="urn:adsk.eagle:library:217" deviceset="LED_E" device="" package3d_urn="urn:adsk.eagle:package:13319/1"/>
+<part name="LED2" library="eagle-ltspice" library_urn="urn:adsk.eagle:library:217" deviceset="LED_E" device="" package3d_urn="urn:adsk.eagle:package:13319/1"/>
 <part name="GND3" library="supply1" library_urn="urn:adsk.eagle:library:371" deviceset="GND" device=""/>
 <part name="GND4" library="supply1" library_urn="urn:adsk.eagle:library:371" deviceset="GND" device=""/>
@@
 <part name="GND10" library="supply1" library_urn="urn:adsk.eagle:library:371" deviceset="GND" device=""/>
 <part name="GND11" library="supply1" library_urn="urn:adsk.eagle:library:371" deviceset="GND" device=""/>
+<part name="+3V4" library="supply1" library_urn="urn:adsk.eagle:library:371" deviceset="+3V3" device=""/>
+<part name="JP6" library="jumper" library_urn="urn:adsk.eagle:library:252" deviceset="JP1Q" device="" package3d_urn="urn:adsk.eagle:package:15455/1"/>
 </parts>
 <sheets>
@@
 <instance part="R10" gate="G$1" x="30.48" y="27.94" rot="R270"/>
 <instance part="+3V10" gate="G$1" x="40.64" y="12.7"/>
-<instance part="LED3" gate="G$1" x="68.58" y="7.62"/>
-<instance part="LED4" gate="G$1" x="81.28" y="7.62"/>
+<instance part="LED1" gate="G$1" x="68.58" y="7.62"/>
+<instance part="LED2" gate="G$1" x="81.28" y="7.62"/>
 <instance part="GND3" gate="1" x="68.58" y="-2.54"/>
 <instance part="GND4" gate="1" x="81.28" y="-2.54"/>
@@
 <instance part="GND1" gate="1" x="2.54" y="33.02"/>
 <instance part="GND2" gate="1" x="2.54" y="-10.16"/>
-<instance part="+3V1" gate="G$1" x="-15.24" y="15.24"/>
+<instance part="+3V1" gate="G$1" x="-5.08" y="-15.24"/>
 <instance part="+3V2" gate="G$1" x="38.1" y="55.88"/>
-<instance part="JP5" gate="A" x="-15.24" y="0"/>
+<instance part="JP5" gate="A" x="-5.08" y="-30.48"/>
 <instance part="CON1" gate="-1" x="12.7" y="22.86" rot="R180"/>
 <instance part="CON1" gate="-2" x="12.7" y="20.32" rot="R180"/>
 <instance part="CON1" gate="-3" x="12.7" y="17.78" rot="R180"/>
-<instance part="CON1" gate="-TABS" x="-12.7" y="-15.24" rot="R180"/>
+<instance part="CON1" gate="-TABS" x="-17.78" y="5.08" rot="R180"/>
 <instance part="CON1" gate="-4" x="12.7" y="15.24" rot="R180"/>
 <instance part="CON2" gate="-1" x="12.7" y="-20.32" rot="R180"/>
 <instance part="CON2" gate="-2" x="12.7" y="-22.86" rot="R180"/>
 <instance part="CON2" gate="-3" x="12.7" y="-25.4" rot="R180"/>
-<instance part="CON2" gate="-TABS" x="-12.7" y="-17.78" rot="R180"/>
+<instance part="CON2" gate="-TABS" x="-17.78" y="2.54" rot="R180"/>
 <instance part="CON2" gate="-4" x="12.7" y="-27.94" rot="R180"/>
 <instance part="CON5" gate="-1" x="91.44" y="-15.24" rot="R180"/>
@@
 <instance part="GND10" gate="1" x="-68.58" y="106.68"/>
 <instance part="GND11" gate="1" x="-43.18" y="116.84"/>
+<instance part="+3V4" gate="G$1" x="-7.62" y="33.02"/>
+<instance part="JP6" gate="A" x="-7.62" y="17.78"/>
 </instances>
 <busses>
@@
 <net name="GND" class="0">
 <segment>
-<pinref part="LED3" gate="G$1" pin="C"/>
+<pinref part="LED1" gate="G$1" pin="C"/>
 <pinref part="GND3" gate="1" pin="GND"/>
 <wire x1="68.58" y1="2.54" x2="68.58" y2="0" width="0.1524" layer="91"/>
 </segment>
 <segment>
-<pinref part="LED4" gate="G$1" pin="C"/>
+<pinref part="LED2" gate="G$1" pin="C"/>
 <pinref part="GND4" gate="1" pin="GND"/>
 <wire x1="81.28" y1="2.54" x2="81.28" y2="0" width="0.1524" layer="91"/>
@@
 </segment>
 <segment>
-<pinref part="JP5" gate="A" pin="2"/>
-<pinref part="+3V1" gate="G$1" pin="+3V3"/>
-<wire x1="-15.24" y1="7.62" x2="-15.24" y2="12.7" width="0.1524" layer="91"/>
-</segment>
-<segment>
 <pinref part="J21" gate="A" pin="1"/>
 <pinref part="+3V3" gate="G$1" pin="+3V3"/>
 <wire x1="-60.96" y1="78.74" x2="-68.58" y2="78.74" width="0.1524" layer="91"/>
+</segment>
+<segment>
+<pinref part="JP6" gate="A" pin="2"/>
+<pinref part="+3V4" gate="G$1" pin="+3V3"/>
+<wire x1="-7.62" y1="25.4" x2="-7.62" y2="30.48" width="0.1524" layer="91"/>
+</segment>
+<segment>
+<pinref part="JP5" gate="A" pin="2"/>
+<pinref part="+3V1" gate="G$1" pin="+3V3"/>
+<wire x1="-5.08" y1="-22.86" x2="-5.08" y2="-17.78" width="0.1524" layer="91"/>
 </segment>
 </net>
@@
 <net name="N$3" class="0">
 <segment>
-<pinref part="LED3" gate="G$1" pin="A"/>
+<pinref part="LED1" gate="G$1" pin="A"/>
 <pinref part="R21" gate="G$1" pin="1"/>
 <wire x1="68.58" y1="10.16" x2="68.58" y2="15.24" width="0.1524" layer="91"/>
@@
 <net name="N$4" class="0">
 <segment>
-<pinref part="LED4" gate="G$1" pin="A"/>
+<pinref part="LED2" gate="G$1" pin="A"/>
 <pinref part="R22" gate="G$1" pin="1"/>
 <wire x1="81.28" y1="10.16" x2="81.28" y2="15.24" width="0.1524" layer="91"/>
@@
 <segment>
 <wire x1="12.7" y1="-38.1" x2="-5.08" y2="-38.1" width="0.1524" layer="91"/>
-<wire x1="-5.08" y1="-7.62" x2="12.7" y2="10.16" width="0.1524" layer="91"/>
-<wire x1="12.7" y1="10.16" x2="12.7" y2="15.24" width="0.1524" layer="91"/>
-<wire x1="-5.08" y1="-38.1" x2="-5.08" y2="-7.62" width="0.1524" layer="91"/>
-<pinref part="JP5" gate="A" pin="1"/>
-<wire x1="-15.24" y1="-7.62" x2="-5.08" y2="-7.62" width="0.1524" layer="91"/>
-<junction x="-5.08" y="-7.62"/>
-<pinref part="CON1" gate="-4" pin="S"/>
 <pinref part="CON2" gate="-4" pin="S"/>
 <wire x1="12.7" y1="-38.1" x2="12.7" y2="-27.94" width="0.1524" layer="91"/>
-</segment>
-</net>
+<pinref part="JP5" gate="A" pin="1"/>
+</segment>
+</net>
+<net name="N$5" class="0">
+<segment>
+<pinref part="CON1" gate="-4" pin="S"/>
+<wire x1="12.7" y1="10.16" x2="12.7" y2="15.24" width="0.1524" layer="91"/>
+<pinref part="JP6" gate="A" pin="1"/>
+<wire x1="-7.62" y1="10.16" x2="12.7" y2="10.16" width="0.1524" layer="91"/>
+</segment>
+</net>
