File: communications_hub/communication-hub/communication-hub.sch (EAGLE design)
At the start: 41 parts, among them CON1 SM04B-GHS-TB, CON2 SM04B-GHS-TB, CON3 SM03B-GHS-TB, CON4 SM03B-GHS-TB, CON5 SM02B-GHS-TB, U3 TCAN1042HVDR, U4 TCAN1042HVDR

Commit message: Slightly modified layout+routing
Parts:
- added R1, R2: 10k, resistor:R-EU_R0805
- R15, R16, R18, R19: value 10K -> 220
- R17: value 10K -> 1k
- R20: value 10K -> 1K
Connections:
- net +3V3: now also J21.17, J26.2
- net +5V: now also J21.4, J26.8
- net GND: now also CON1-TABS.S, CON2-TABS.S, CON3-TABS.S, CON4-TABS.S, CON5-TABS.S, J21.39, J26.10, J26.11, J26.21, R1.1, R2.1; no longer J21.35
- net N$27: now also R1.2
- net N$30: now also R2.2
Other:
- moved on the sheet: C10, C11, C12, C7, C8, C9, CON1-1, CON1-2, CON1-3, CON1-4, CON1-TABS, CON2-1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
