File: battery_monitoring_17-18/Battery_Monitoring_with_kill.sch (EAGLE design)
At the start: 53 parts, among them CON4 MOLEX_5566-2, CON5 S3B-PH-SM4-TB, CON6 S3B-PH-SM4-TB, U1 INA3221., U2 INA3221., U4 TEENSY_3.1_BASIC_2, U6 TCAN1042HVDR

Commit message: Changed JST connector; Rearranged folders; Generated CAM files
Parts:
- removed C5, C6: 10u, rcl:C-EUC0805
- removed CON4: MOLEX_5566-2, ARVP:MOLEX_5566-2
- removed CON5, CON6: S3B-PH-SM4-TB, ARVP:S3B-PH-SM4-TB
- removed R22, R23, R24: 10k, adafruit:R-US_M1206
- removed R25, R26, R27: 1k, adafruit:R-US_M1206
- removed U$1, U$2, U$3, U$4, U$5, U$6, U$7, U$8: MKDS_5/2-6,352, Moira:MKDS_5/2-6,352
- removed U$10: ARVP_LOGO, ARVP:ARVP_LOGO
- removed U$11, U$12, U$13: TCLD1000CT, Moira:TCLD1000CT
- removed U$14, U$19, U$20: PSMN1R5-30BLE, Moira:PSMN1R5-30BLE
- removed U$21, U$22, U$23: BZT52C10, Moira:BZT52C10
- removed U6: TCAN1042HVDR, ARVP:TCAN1042HVDR
- added ARVP1: ARVP_LOGO, ARVP:ARVP_LOGO
- added C1: 0.1microF, resistor:C-USC2012
- added C3: 10u, rcl:C-EUC0805
- added CON1: MOLEX_5566-2, ARVP:MOLEX_5566-2
- added CON2, CON3: SM03B-GHS-TB, ARVP:SM03B-GHS-TB
- added D1, D2, D3: BZT52C10, Moira:BZT52C10
- added J1, J2, J3, J4, J5, J6, J7, J8: MKDS_5/2-6,352, Moira:MKDS_5/2-6,352
- added Q1, Q2, Q3: TCLD1000CT, Moira:TCLD1000CT
- added Q4, Q5, Q6: PSMN1R5-30BLE, Moira:PSMN1R5-30BLE
- added R14, R15: 10k, rcl:R-US_R1206
- added R17: 220, rcl:R-US_R0805
- added R18: 1k, rcl:R-US_R0805
- added R2: 1k, adafruit:R-US_R0805
- added R5: 1k, adafruit:R-US_M1206
- added U3: TEENSY_3.1_BASIC_2, Teensy_3_Series_Board_v1.0:TEENSY_3.1_BASIC_2
- C4: value 0.1microF -> 10u; device resistor:C-USC2012 -> rcl:C-EUC0805
- JP1: device pinhead:PINHD-2X3 -> pinhead:PINHD-1X2
- JP2: device pinhead:PINHD-1X2 -> pinhead:PINHD-1X3
- JP3: device pinhead:PINHD-2X4 -> pinhead:PINHD-1X2
- JP5: device pinhead:PINHD-1X2 -> pinhead:PINHD-2X3
- JP6: device pinhead:PINHD-1X3 -> pinhead:PINHD-2X4
- R1, R3: value 0.001Ohm -> 1k; device Moira:HCS3920FT1L00 -> adafruit:R-US_R0805
- R10, R9: device rcl:R-US_R1206 -> adafruit:R-US_M1206
- R11: value 1k -> 10k; device adafruit:R-US_R0805 -> adafruit:R-US_M1206
- R12, R13: value 1k -> 0.001Ohm; device adafruit:R-US_R0805 -> Moira:HCS3920FT1L00
- R16: value 1k -> 220
- R6: value 220 -> 1k; device rcl:R-US_R0805 -> adafruit:R-US_M1206
- R7: value 0.001Ohm -> 1k; device Moira:HCS3920FT1L00 -> adafruit:R-US_M1206
- R8: value 220 -> 0.001Ohm; device rcl:R-US_R0805 -> Moira:HCS3920FT1L00
- U4: value TEENSY_3.1_BASIC_2 -> TCAN1042HVDR; device Teensy_3_Series_Board_v1.0:TEENSY_3.1_BASIC_2 -> ARVP:TCAN1042HVDR
Connections:
- net +3V3: now also C1.1, C3.1, JP5.1, JP5.3, JP5.5, U3.3.3V, U4.VIO; no longer C4.1, C5.1, JP1.1, JP1.3, JP1.5, U4.3.3V, U6.VIO
- net +5V: now also CON1G$1.S, JP2.1, JP4.2, R1.1, R2.1, R3.1; no longer CON4G$1.S, JP2.2, JP6.1, R11.1, R12.1, R13.1
- net 0-26V_BATTERY1: now also J4.KL, Q1.C2, R8.2; no longer R4.2, U$1.KL, U$11.C2
- net 0-26V_BATTERY2: now also J3.KL, Q2.C2, R4.2; no longer R1.2, U$12.C2, U$2.KL
- net 0-26V_BATTERY3: now also J2.KL, Q3.C2, R13.2; no longer R3.2, U$13.C2, U$3.KL
- net 0-26V_BATTERY4: now also J1.KL, R12.2; no longer R7.2, U$4.KL
- net CANH1: now also CON2-3.S, CON3-3.S, U4.CANH; no longer CON5-3.S, CON6-3.S, U6.CANH
- net CANL1: now also CON2-2.S, CON3-2.S, U4.CANL; no longer CON5-2.S, CON6-2.S, U6.CANL
- net CANSH1: now also CON2-1.S, CON3-1.S; no longer CON5-1.S, CON6-1.S
- net CAN_RX1: now also R17.2, U4.RXD; no longer R8.2, U6.RXD
- net CAN_RX_T: now also R17.1, U3.4/CAN-RX-PWM; no longer R8.1, U4.4/CAN-RX-PWM
- net CAN_TX2: now also R16.2, U4.TXD; no longer R6.2, U6.TXD
- net CAN_TX_T: now also R16.1, U3.3/CAN-TX/PWM; no longer R6.1, U4.3/CAN-TX/PWM
- net CRITICAL_OUT: now also U3.9/RX2/PWM; no longer U4.9/RX2/PWM
- net E1: now also Q1.E, R5.2; no longer R25.2, U$11.E
- net E2: now also Q2.E, R6.2; no longer R26.2, U$12.E
- net E3: now also Q3.E, R7.2; no longer R27.2, U$13.E
- net GND: now also C1.2, C3.2, CON1G$2.S, CON2-TABS.S, CON3-TABS.S, D1.A, D2.A, D3.A, J1.KL1, J2.KL1, J3.KL1, J4.KL1, J8.KL1, JP1.2, JP2.3, JP6.1, JP6.2, Q4.S, Q5.S, Q6.S, R10.1, R11.1, R18.1, R9.1, U3.GND; no longer C5.2, C6.2, CON4G$2.S, CON5-TABS.S, CON6-TABS.S, JP3.1, JP3.2, JP4.2, JP6.3, R16.1, R22.1, R23.1, R24.1, U$1.KL1, U$14.S, U$19.S, U$2.KL1, U$20.S, U$21.A, U$22.A, U$23.A, U$3.KL1, U$4.KL1, U$8.KL1, U6.GND
- net I2C_3V1: now also JP5.6, JP6.7, JP6.8; no longer JP1.6, JP3.7, JP3.8
- net MD1: now also J5.KL1, Q4.D; no longer U$14.D, U$5.KL1
- net MD2: now also J6.KL1, Q5.D; no longer U$19.D, U$6.KL1
- net MD3: now also J7.KL1, Q6.D; no longer U$20.D, U$7.KL1
- net MG1: now also D1.C, Q4.G, R5.1, R9.2; no longer R22.2, R25.1, U$14.G, U$21.C
- net MG2: now also D2.C, Q5.G, R10.2, R6.1; no longer R23.2, R26.1, U$19.G, U$22.C
- net MG3: now also D3.C, Q6.G, R11.2, R7.1; no longer R24.2, R27.1, U$20.G, U$23.C
- net MOTOR1: now also J5.KL, R8.1; no longer R4.1, U$5.KL
- net MOTOR2: now also J6.KL, R4.1; no longer R1.1, U$6.KL
- net MOTOR3: now also J7.KL, R13.1; no longer R3.1, U$7.KL
- net MOTOR4: now also J8.KL, R12.1; no longer R7.1, U$8.KL
- net N$1: now also Q1.A, R1.2; no longer R11.2, U$11.A
- net N$2: now also Q2.A, R2.2; no longer R12.2, U$12.A
- net N$3: now also Q3.A, R3.2; no longer R13.2, U$13.A
- net N$4: now also JP1.1, JP3.1, Q1.C1, Q2.C1, Q3.C1; no longer JP4.1, JP5.1, U$11.C1, U$12.C1, U$13.C1
- net N$5: now also JP2.2, JP3.2; no longer JP5.2, JP6.2
- net PV_OUT: now also U3.7/RX3; no longer U4.7/RX3
- net SCL: now also JP6.5, JP6.6, R14.2, U3.19/A5/T/SCL0; no longer JP3.5, JP3.6, R10.2, U4.19/A5/T/SCL0
- net SCL_3V1: now also JP5.2, R14.1; no longer JP1.2, R10.1
- net SDA: now also JP6.3, JP6.4, R15.2, U3.18/A4/T/SDA0; no longer JP3.3, JP3.4, R9.2, U4.18/A4/T/SDA0
- net SDA_3V1: now also JP5.4, R15.1; no longer JP1.4, R9.1
- net STB1: now also R18.2, U4.STB; no longer R16.2, U6.STB
- net TC_OUT: now also U3.8/TX3; no longer U4.8/TX3
- net VIN: now also C4.1, JP4.1, U3.VIN, U4.VCC; no longer C6.1, JP2.1, U4.VIN, U6.VCC
- net WARNING_OUT: now also U3.10/TX2/PWM; no longer U4.10/TX2/PWM
Other:
- moved on the sheet: C2, C4, JP4, R1, R10, R11, R12, R13, R16, R3, R4, R6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

Commit message: Fixed issue where motors could still find ground return path even when battery was disconnected by mosfet
Connections:
- removed net MD1: J5.KL1, Q4.D
- removed net MD2: J6.KL1, Q5.D
- removed net MD3: J7.KL1, Q6.D
- new net BATT1GND: D1.A, J4.KL, Q4.S, R9.1
- new net BATT2GND: D2.A, J3.KL, Q5.S, R10.1
- new net BATT3GND: D3.A, J2.KL, Q6.S, R11.1
- net 0-26V_BATTERY1: now also J4.KL1; no longer J4.KL
- net 0-26V_BATTERY2: now also J3.KL1; no longer J3.KL
- net 0-26V_BATTERY3: now also J2.KL1; no longer J2.KL
- net 0-26V_BATTERY4: now also J1.KL1; no longer J1.KL
- net GND: now also J1.KL, J5.KL1, J6.KL1, J7.KL1, Q4.D, Q5.D, Q6.D; no longer D1.A, D2.A, D3.A, J1.KL1, J2.KL1, J3.KL1, J4.KL1, Q4.S, Q5.S, Q6.S, R10.1, R11.1, R9.1
Other:
- moved on the sheet: CON1G$1, CON1G$2, J1, J2, J3, J4
