File: sonar/preprocessor_v3/design_blocks/Amplifier-Sonar - ARVP/Design Block/Three Amplifier Block/Alternative Design/Sonar-Three-Amp-Block.brd (EAGLE design)
At the start: 16.4 x 40 mm, 36 parts, among them U1 ISL21080DIH309Z-TK, U2 AD8336ACPZ-R7, U4 AD8336ACPZ-R7, U6 AD8336ACPZ-R7

Commit message: Routing and layout work
Parts:
- moved C22 6.56 mm to (16.6, 9.35), turned to 90 degrees
- moved C34 5.74 mm to (16.6, 20.7), turned to 90 degrees
- moved C10 5.74 mm to (16.6, 32.0), turned to 90 degrees
- moved C1 2.04 mm to (10.1, 5.78)
- moved C3 2.04 mm to (10.1, 3.73)
- moved U1 1.91 mm to (13.5, 4.91)
Routing:
- net GAIN_NEG: track 26.6 -> 39.3 mm, vias 3 -> 4
- net -5V: track 14.9 -> 7.59 mm
- removed copper zone on layer 1, net GND
Other:
- board outline removed
