File: wiring_diagrams/Wiring Diagrams.sch (EAGLE design)
At the start: 0 parts

Commit message: Added proper paging and most power diagrams
Other:
- note added: "+12V GND"
- note added: "+5V CANH CANL SHIELD"
- note added: "+5V GND"
- note added: "120 Ohm Term"
- note added: "Barrel"
- note added: "CAN0 Bus"
- note added: "CAN1 Bus"
- note added: "CAN2"
- note added: "CANH CANL SHIELD"
- note added: "Comm Board"
- note added: "ESC CAN layout"
- note added: "GND +5V"
- note added: "Top Bottom"
- note added: "USB, Eth, and UART"
- note removed: "120 Ohm Split Term"
- note removed: "CANH CANL GND"
- note removed: "P. 1/5"
- note removed: "P. 2/5"
- note removed: "P. 3/5"
- note removed: "P. 4/5"
- note removed: "P. 5/5"
- note removed: "USB, Ethernet, and UART"

Commit message: Updated diagrams
Other:
- note added: "DVL- 1000"
- note added: "DVL-1000"
- note added: "SHIELD CANL CANH"
- note added: "SHIELD CANL CANH +5V"
- note removed: "+5V CANH CANL GND"
- note removed: "CANH CANL SHIELD"
- note removed: "TX RX"
- note removed: "UART"
