File: battery_monitoring_board/V2_2018_2019/Battery_BoardV2/Battery_Monitoring_V2.sch (EAGLE design)
At the start: 83 parts, among them CON1 MOLEX_5566-2, CON2 SM03B-GHS-TB, CON3 SM03B-GHS-TB, J1 MKDS_5/2-6,352, J2 MKDS_5/2-6,352, J3 MKDS_5/2-6,352, J4 MKDS_5/2-6,352, J5 MKDS_5/2-6,352, J6 MKDS_5/2-6,352, J7 MKDS_5/2-6,352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

Commit message: PCB is done except for DRC, BOM is done
Parts:
- C10, C5, C6, C7, C8, C9: device adafruit:C-USC1206 -> adafruit:C-USC0805
- R23, R24, R26, R27, R28, R29, R30: device adafruit:R-US_R1206 -> adafruit:R-US_R0805
