File: sonar/preprocessor_v5/sonar_preprocessor.brd (EAGLE design)
At the start: 130.8 x 68.6 mm, 217 parts, among them CON4 MOLEX_5566-2, J1 TE_5-1634503-1TE, J2 TE_5-1634503-1TE, J3 TE_5-1634503-1TE, J4 TE_5-1634503-1TE, U1 TEENSY_3.1_BASIC, U10 LT1117-5, U11 MMBT3904, U12 AD8336ACPZ-R7, U13 AD8336ACPZ-R7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

Commit message: completed routing
Parts:
- moved CON4 17.8 mm to (72.4, 52.6)
- moved R10 6.35 mm to (117.7, 90.6)
- moved R38 6.35 mm to (119.9, 84.2)
- moved R39 6.35 mm to (117.7, 84.2)
- moved R9 6.35 mm to (119.9, 90.6)
- moved C10 6.35 mm to (124.7, 91.4)
- moved C68 6.35 mm to (124.7, 85.1)
- moved R11 6.35 mm to (118.9, 93.7)
- moved R40 6.35 mm to (118.9, 87.4)
- moved TP13 6.35 mm to (130.2, 85.1)
- moved TP9 6.35 mm to (130.2, 91.4)
- moved TP7 3.05 mm to (130.2, 107.2)
- moved H4 0.25 mm to (186.4, 49.5)
- turned R1C2 to 0 degrees
Connections:
- net INPUT3: no longer U19.2
- net INPUT4: now also U19.2
Routing:
- net GAIN_POS: track 93.8 -> 136.7 mm, vias 5 -> 6
- net AMP_4: track 0.00 -> 39.5 mm
- net INPUT4: track 0.00 -> 30.2 mm
- net N$8: track 0.00 -> 29.2 mm
- net V+: track 23.4 -> 47.5 mm
- net GAIN_NEG: track 39.3 -> 61.3 mm, vias 4 -> 5
- net SIG_OUT_3: track 0.00 -> 20.6 mm
- net CLAMP_IN_3: track 0.00 -> 19.3 mm, vias 0 -> 2
- net OUT_2ND_B2: track 0.00 -> 19.1 mm
- net GPIO_2: track 0.00 -> 17.7 mm
- net GPIO_0: track 0.00 -> 17.7 mm
- net GPIO_1: track 0.00 -> 17.7 mm
- net FILTER_OUT_4: track 0.00 -> 16.7 mm
- net GPIO_3: track 0.00 -> 16.6 mm
- net SIG_OUT_2: track 22.2 -> 37.2 mm
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
Commit message: minor changes
Routing:
- net N$14: track 4.64 -> 3.81 mm
Other:
- board text added: "CREDIT: NICHOLAS K. MOIRA B. KOLTIN K.-H. DAVID L. ALAIN L. Andrew S. Kirill M."
- board text added: "HYDROPHONE SIGNAL PROCESSOR V5 Rev. 1: 05/2020"
- board text removed: "CREDIT: NICHOLAS K. MOIRA B. KOLTIN K.-H. DAVID L. ALAIN L. Andrew S."
- board text removed: "HYDROPHONE SIGNAL PROCESSOR V4 Rev. 1: 11/2018"
Changed lines of the file:
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@@
 REFS</text>
 <text x="85.09" y="107.95" size="1.4224" layer="21" align="top-left">HYDROPHONE SIGNAL
-PROCESSOR V4
-Rev. 1: 11/2018</text>
-<text x="69.85" y="99.06" size="1.4224" layer="21">CREDIT:
+PROCESSOR V5
+Rev. 1: 05/2020</text>
+<text x="69.85" y="97.79" size="1.4224" layer="21">CREDIT:
 NICHOLAS K.
 MOIRA B.
@@
 DAVID L.
 ALAIN L.
-Andrew S.</text>
+Andrew S.
+Kirill M.</text>
 <text x="1.27" y="-48.26" size="1.4224" layer="21"></text>
 <text x="137.16" y="69.85" size="1.27" layer="21" rot="R90" align="center-left">12</text>
@@
 <dimension x1="193.04" y1="44.45" x2="199.39" y2="44.45" x3="196.215" y3="41.91" textsize="1.778" layer="47" dtype="horizontal" unit="inch" visible="yes"/>
 <text x="197.104" y="81.788" size="1.27" layer="21" rot="R180">GND</text>
+<dimension x1="57.15" y1="115.57" x2="57.15" y2="46.99" x3="59.69" y3="81.28" textsize="1.778" layer="47"/>
 </plain>
 <attributes>
@@
 <via x="107.95" y="96.52" extent="1-16" drill="0.3"/>
 <via x="109.855" y="95.25" extent="1-16" drill="0.3"/>
-<via x="113.665" y="94.234" extent="1-16" drill="0.3"/>
+<via x="113.284" y="94.0308" extent="1-16" drill="0.3"/>
 <via x="115.9256" y="106.0704" extent="1-16" drill="0.3"/>
 <via x="120.015" y="109.22" extent="1-16" drill="0.3"/>
@@
 <contactref element="D4" pad="1"/>
 <contactref element="U6" pad="2"/>
-<wire x1="112.225" y1="96.332" x2="113.157" y2="93.957" width="0.2032" layer="1"/>
-<wire x1="113.157" y1="93.957" x2="113.157" y2="92.136" width="0.2032" layer="1"/>
 <wire x1="113.157" y1="92.136" x2="110.175" y2="92.136" width="0.2032" layer="1"/>
 <wire x1="110.175" y1="92.136" x2="109.728" y2="92.583" width="0.2032" layer="1"/>
 <wire x1="109.728" y1="92.583" x2="109.728" y2="93.8784" width="0.2032" layer="1"/>
+<wire x1="112.225" y1="96.332" x2="112.225" y2="93.068" width="0.2032" layer="1"/>
+<wire x1="112.225" y1="93.068" x2="113.157" y2="92.136" width="0.2032" layer="1"/>
 </signal>
 <signal name="PEAK_OUT">
@@
 <contactref element="D4" pad="3"/>
 <contactref element="U6" pad="1"/>
-<wire x1="110.025" y1="97.282" x2="111.717" y2="96.223" width="0.2032" layer="1"/>
-<wire x1="111.717" y1="96.223" x2="110.998" y2="95.504" width="0.2032" layer="1"/>
 <wire x1="110.998" y1="95.504" x2="110.998" y2="93.8784" width="0.2032" layer="1"/>
+<wire x1="110.025" y1="97.282" x2="110.025" y2="96.477" width="0.2032" layer="1"/>
+<wire x1="110.025" y1="96.477" x2="110.998" y2="95.504" width="0.2032" layer="1"/>
 </signal>
 <signal name="PEAK_CLEAR">
@@
 <wire x1="171.069" y1="50.0634" x2="169.2656" y2="48.26" width="0.254" layer="16"/>
 <wire x1="169.2656" y1="48.26" x2="148.59" y2="48.26" width="0.254" layer="16"/>
-<via x="167.83" y="62.1102" extent="1-16" drill="0.35"/>
-<wire x1="167.805" y1="61.7352" x2="167.461709375" y2="61.98365625" width="0.254" layer="1"/>
-<wire x1="167.461709375" y1="61.98365625" x2="166.7002" y2="62.5348" width="0.254" layer="1"/>
+<via x="167.83" y="62.288" extent="1-16" drill="0.35"/>
 <wire x1="135.89" y1="71.12" x2="133.35" y2="73.66" width="0.254" layer="1"/>
 <wire x1="143.51" y1="71.12" x2="135.89" y2="71.12" width="0.254" layer="1"/>
-<wire x1="167.805" y1="60.3393" x2="167.805" y2="61.7352" width="0.254" layer="1"/>
-<wire x1="166.7002" y1="62.5348" x2="166.7002" y2="63.2738" width="0.254" layer="1"/>
-<wire x1="166.7002" y1="63.2738" x2="166.28" y2="63.694" width="0.254" layer="1"/>
-<wire x1="167.83" y1="62.1102" x2="167.83" y2="73.66" width="0.254" layer="15"/>
-<wire x1="169.799" y1="60.1412" x2="167.83" y2="62.1102" width="0.254" layer="15"/>
-<wire x1="167.461709375" y1="61.98365625" x2="167.70345625" y2="61.98365625" width="0.254" layer="1"/>
-<wire x1="167.70345625" y1="61.98365625" x2="167.83" y2="62.1102" width="0.254" layer="1"/>
+<wire x1="167.83" y1="62.288" x2="167.83" y2="73.66" width="0.254" layer="15"/>
+<wire x1="169.799" y1="60.1412" x2="167.83" y2="62.288" width="0.254" layer="15"/>
 <wire x1="171.069" y1="55.118" x2="170.5356" y2="55.118" width="0.254" layer="15"/>
 <wire x1="170.5356" y1="55.118" x2="169.799" y2="55.8546" width="0.254" layer="15"/>
+<wire x1="167.805" y1="60.3393" x2="167.805" y2="62.263" width="0.254" layer="1"/>
+<wire x1="167.805" y1="62.263" x2="167.83" y2="62.288" width="0.254" layer="1"/>
+<wire x1="167.83" y1="62.288" x2="167.686" y2="62.288" width="0.254" layer="1"/>
+<wire x1="167.686" y1="62.288" x2="166.28" y2="63.694" width="0.254" layer="1"/>
 </signal>
 <signal name="INPUT1">
