File: Actuator_board/dropper_torpedo trail 2.brd (EAGLE design)
At the start: 76.2 x 50.8 mm, 72 parts, among them CON1 SM03B-GHS-TB, CON2 SM03B-GHS-TB, CON3 MOLEX_5566-2, CON4 MOLEX_5566-2, CON6 MOLEX_5566-2, Q1 SI4896DY-T1-E3, Q2 SI4896DY-T1-E3, Q3 IRL6372TRPBF, Q4 IRL6372TRPBF, U1 LTV-355T, U2 LTV-355T, U3 TCAN1042HVDR, U4 PCA9685PW, U5 TEENSY_3.1_BASIC_2, X1 OSTVN05A150, X2 MOLEX_5566-4

Commit message: Removed components
Parts:
- removed C1, C2: 1u, rcl:C1206
- removed CON4, CON6: MOLEX_5566-2, ARVP:5566-2
- removed D1, D2: STPS1L30A, dropper_torpedo_v3:DO214AC
- removed JP10: (no value), pinhead:2X06
- removed JP8: (no value), pinhead:2X04
- removed JP9: (no value), pinhead:2X03
- removed LED1, LED2: (no value), led:CHIPLED_1206
- removed Q1, Q2: SI4896DY-T1-E3, dropper_torpedo_v3:SO-8
- removed R1, R2: 3k, rcl:R1206
- removed R10, R11, R12, R9: 5k, rcl:R0805
- removed R20, R21, R3, R4: 10k, rcl:R1206
- removed R22: 10k, ARVP:EXBV8V-M
- removed R5, R6: 1k, rcl:R1206
- removed R7, R8: 2k, rcl:R1206
- removed U1, U2: LTV-355T, dropper_torpedo_v3:SMD4
Connections:
- removed net A0: R26.6, U4.1
- removed net A0+: JP10.2, R26.3
- removed net A1: R26.5, U4.2
- removed net A1+: JP10.4, R26.4
- removed net A2: R22.8, U4.3
- removed net A2+: JP10.6, R22.1
- removed net A3: R22.7, U4.4
- removed net A3+: JP10.8, R22.2
- removed net A4: R22.6, U4.5
- removed net A4+: JP10.10, R22.3
- removed net A5: R22.5, U4.24
- removed net A5+: JP10.12, R22.4
- removed net I2C_3V3: JP8.7, JP8.8, JP9.6
- removed net N$1: LED1.A, R7.1
- removed net N$2: LED2.A, R8.1
- removed net RC0: C1.2, R1.2
- removed net RC1: C2.2, R2.2
- removed net SCL: JP8.5, JP8.6, R20.2, U4.26, U5.19/A5
- removed net SCL_3V3: JP9.2, R20.1
- removed net SDA: JP8.3, JP8.4, R21.2, U4.27, U5.18/A4
- removed net SDA_3V3: JP9.4, R21.1
- removed net TOPTO_A0: R10.1, R9.1, U1.ANODE
- removed net TOPTO_A1: R11.1, R12.1, U2.ANODE
- removed net TOPTO_E0: R5.2, R7.2, U1.EMITTER
- removed net TOPTO_E1: R6.2, R8.2, U2.EMITTER
- removed net TRP0: R10.2, U5.16/A2
- removed net TRP0_ALT: JP7.4, R9.2
- removed net TRP1: R12.2, U5.17/A3
- removed net TRP1_ALT: JP7.2, R11.2
- removed net TRP_GATE0: Q1.4, R3.2, R5.1
- removed net TRP_GATE1: Q2.4, R4.2, R6.1
- removed net TRP_RETURN0: C1.1, D1.A, Q1.5, Q1.6, Q1.7, Q1.8
- removed net TRP_RETURN1: C2.1, D2.A, Q2.5, Q2.6, Q2.7, Q2.8
- net +12V: no longer CON4.1, CON4.2, CON6.1, CON6.2, D1.C, D2.C, U1.COLLECTOR, U2.COLLECTOR
- net +3V3: no longer JP10.1, JP10.11, JP10.3, JP10.5, JP10.7, JP10.9, JP9.1, JP9.3, JP9.5
- net GND: no longer JP8.1, JP8.2, LED1.C, LED2.C, Q1.1, Q1.2, Q1.3, Q2.1, Q2.2, Q2.3, R1.1, R2.1, R3.1, R4.1, U1.CATHODE, U2.CATHODE
Routing:
- net SCL: track 54.0 -> 0.00 mm, vias 2 -> 0
- net SDA: track 50.2 -> 0.00 mm, vias 2 -> 0
- net TOPTO_E0: track 45.3 -> 0.00 mm
- net TRP0_ALT: track 41.6 -> 0.00 mm, vias 2 -> 0
- net TRP1_ALT: track 36.8 -> 0.00 mm
- net +12V: track 37.0 -> 5.04 mm
- net TOPTO_E1: track 26.8 -> 0.00 mm, vias 2 -> 0
- net I2C_3V3: track 19.7 -> 0.00 mm
- net TRP0: track 19.1 -> 0.00 mm
- net TRP1: track 15.3 -> 0.00 mm
- net A5: track 14.1 -> 0.00 mm, vias 2 -> 0
- net TRP_GATE0: track 12.1 -> 0.00 mm
- net TRP_GATE1: track 11.9 -> 0.00 mm
- net +3V3: track 105.8 -> 96.7 mm
- net TRP_RETURN0: track 7.89 -> 0.00 mm
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- removed copper zone on layer 16, net +12V
- removed copper zone on layer 1, net TRP_RETURN0
- removed copper zone on layer 1, net TRP_RETURN1
Other:
- board text removed: "I2C"
- board text removed: "I2C CONFIG"
- board text removed: "I2C PWR"
- board text removed: "SCL"
- board text removed: "SDA"
- board text removed: "SWITCH"
- board text removed: "TORPEDO0"
- board text removed: "TORPEDO1"
