File: Actuator_board/dropper_torpedo trail 2.sch (EAGLE design)
At the start: 65 parts, among them CON1 SM03B-GHS-TB, CON2 SM03B-GHS-TB, CON3 MOLEX_5566-2, CON4 MOLEX_5566-2, CON6 MOLEX_5566-2, Q1 SI4896DY-T1-E3, Q2 SI4896DY-T1-E3, Q3 IRL6372TRPBF, Q4 IRL6372TRPBF, U1 LTV-355T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

Commit message: Removed components
Parts:
- removed C1, C2: 1u, rcl:C-EUC1206
- removed CON4, CON6: MOLEX_5566-2, ARVP:MOLEX_5566-2
- removed D1, D2: STPS1L30A, dropper_torpedo_v3:STPS1L30A
- removed JP10: (no value), pinhead:PINHD-2X6
- removed JP8: (no value), pinhead:PINHD-2X4
- removed JP9: (no value), pinhead:PINHD-2X3
- removed LED1, LED2: (no value), led:LEDCHIPLED_1206
- removed Q1, Q2: SI4896DY-T1-E3, dropper_torpedo_v3:SI4896DY-T1-E3
- removed R1, R2: 3k, rcl:R-US_R1206
- removed R10, R11, R12, R9: 5k, rcl:R-US_R0805
- removed R20, R21, R3, R4: 10k, rcl:R-US_R1206
- removed R22: 10k, ARVP:EXB-V8V221JVEXBV8V-M
- removed R5, R6: 1k, rcl:R-US_R1206
- removed R7, R8: 2k, rcl:R-US_R1206
- removed U1, U2: LTV-355T, dropper_torpedo_v3:LTV-355T
Connections:
- removed net A0: R26.66, U4.A0
- removed net A0+: JP10.2, R26.35
- removed net A1: R26.58, U4.A1
- removed net A1+: JP10.4, R26.47
- removed net A2: R22.82, U4.A2
- removed net A2+: JP10.6, R22.11
- removed net A3: R22.74, U4.A3
- removed net A3+: JP10.8, R22.23
- removed net A4: R22.66, U4.A4
- removed net A4+: JP10.10, R22.35
- removed net A5: R22.58, U4.A5
- removed net A5+: JP10.12, R22.47
- removed net I2C_3V3: JP8.7, JP8.8, JP9.6
- removed net N$1: LED1.A, R7.1
- removed net N$2: LED2.A, R8.1
- removed net RC0: C1.2, R1.2
- removed net RC1: C2.2, R2.2
- removed net SCL: JP8.5, JP8.6, R20.2, U4.SCL, U5.19/A5/T/SCL0
- removed net SCL_3V3: JP9.2, R20.1
- removed net SDA: JP8.3, JP8.4, R21.2, U4.SDA, U5.18/A4/T/SDA0
- removed net SDA_3V3: JP9.4, R21.1
- removed net TOPTO_A0: R10.1, R9.1, U1.A
- removed net TOPTO_A1: R11.1, R12.1, U2.A
- removed net TOPTO_E0: R5.2, R7.2, U1.EMIT
- removed net TOPTO_E1: R6.2, R8.2, U2.EMIT
- removed net TRP0: R10.2, U5.16/A2/T
- removed net TRP0_ALT: JP7.4, R9.2
- removed net TRP1: R12.2, U5.17/A3/T
- removed net TRP1_ALT: JP7.2, R11.2
- removed net TRP_GATE0: Q1.G, R3.2, R5.1
- removed net TRP_GATE1: Q2.G, R4.2, R6.1
- removed net TRP_RETURN0: C1.1, D1.A, Q1.D
- removed net TRP_RETURN1: C2.1, D2.A, Q2.D
- net +12V: no longer CON4G$1.S, CON4G$2.S, CON6G$1.S, CON6G$2.S, D1.C, D2.C, U1.COL, U2.COL
- net +3V3: no longer JP10.1, JP10.11, JP10.3, JP10.5, JP10.7, JP10.9, JP9.1, JP9.3, JP9.5
- net GND: no longer JP8.1, JP8.2, LED1.C, LED2.C, Q1.S, Q2.S, R1.1, R2.1, R3.1, R4.1, U1.C, U2.C
